File: learn/udemy/udemy.kicad_sch (KiCad schematic)
At the start: 13 parts, among them J1 Screw_Terminal_01x02, J2 Screw_Terminal_01x02, J3 Screw_Terminal_01x02, U1 L7809, U2 L7805

Commit message: 03/01/23 tutorial comandi menù
Connections:
- net 9v out: now reaches C3.1, D1.2 (A), J2.1 (Pin_1), U1.3 (OUT)
Other:
- note added: "Connettori"
- note added: "Regolatore di tensione"
- moved on the sheet: J1, J2, J3

Commit message: 05/01/23 modifiche al circuito elettrico
Parts:
- C1, C2: value 0.33uF -> 0.50uF
Other:
- note added: "Indicazione LED"
- moved on the sheet: C1, C2, C3, C4, D1, D2, J1, J2, J3, R1, R2, U1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

Commit message: 06/01/23 assegnazione footprint
Parts:
- C1: value 0.50uF -> 0.33uF; footprint (none) -> Resistor_THT:R_Axial_DIN0207_L6.3mm_D2.5mm_P2.54mm_Vertical
- C2: value 0.50uF -> 0.33uF; footprint (none) -> Capacitor_THT:C_Disc_D4.7mm_W2.5mm_P5.00mm
- C3, C4: footprint (none) -> Capacitor_THT:C_Disc_D3.0mm_W2.0mm_P2.50mm
- D1, D2: footprint (none) -> LED_THT:LED_D4.0mm
- J1, J2, J3: footprint (none) -> TerminalBlock_Phoenix:TerminalBlock_Phoenix_MKDS-1,5-2-5.08_1x02_P5.08mm_Horizontal
- R1: footprint (none) -> Resistor_THT:R_Axial_DIN0204_L3.6mm_D1.6mm_P5.08mm_Horizontal
- R2: value R -> 1kohm; footprint (none) -> Resistor_THT:R_Axial_DIN0207_L6.3mm_D2.5mm_P7.62mm_Horizontal
- U1, U2: footprint (none) -> Package_TO_SOT_THT:TO-220-3_Vertical
Changed lines of the file:
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@@
     (property "Reference" "D2" (id 0) (at 107.95 104.4575 0))
     (property "Value" "LED" (id 1) (at 110.49 104.4575 0))
-    (property "Footprint" "" (id 2) (at 114.3 102.87 0)
+    (property "Footprint" "LED_THT:LED_D4.0mm" (id 2) (at 114.3 102.87 0)
       (effects (font (size 1.27 1.27)) hide)
     )
@@
     (property "Reference" "U1" (id 0) (at 99.06 40.64 0))
     (property "Value" "L7809" (id 1) (at 99.06 43.18 0))
-    (property "Footprint" "" (id 2) (at 99.695 52.07 0)
+    (property "Footprint" "Package_TO_SOT_THT:TO-220-3_Vertical" (id 2) (at 99.695 52.07 0)
       (effects (font (size 1.27 1.27) italic) (justify left) hide)
     )
@@
       (effects (font (size 1.27 1.27)) (justify left))
     )
-    (property "Footprint" "" (id 2) (at 208.28 100.33 0)
+    (property "Footprint" "TerminalBlock_Phoenix:TerminalBlock_Phoenix_MKDS-1,5-2-5.08_1x02_P5.08mm_Horizontal" (id 2) (at 208.28 100.33 0)
       (effects (font (size 1.27 1.27)) hide)
     )
@@
       (effects (font (size 1.27 1.27)) (justify left))
     )
-    (property "Footprint" "" (id 2) (at 112.522 114.3 90)
+    (property "Footprint" "Resistor_THT:R_Axial_DIN0204_L3.6mm_D1.6mm_P5.08mm_Horizontal" (id 2) (at 112.522 114.3 90)
       (effects (font (size 1.27 1.27)) hide)
     )
@@
     (property "Reference" "U2" (id 0) (at 135.89 40.64 0))
     (property "Value" "L7805" (id 1) (at 135.89 43.18 0))
-    (property "Footprint" "" (id 2) (at 136.525 52.07 0)
+    (property "Footprint" "Package_TO_SOT_THT:TO-220-3_Vertical" (id 2) (at 136.525 52.07 0)
       (effects (font (size 1.27 1.27) italic) (justify left) hide)
     )
@@
       (effects (font (size 1.27 1.27)) (justify left))
     )
-    (property "Value" "0.50uF" (id 1) (at 92.71 62.2299 0)
-      (effects (font (size 1.27 1.27)) (justify left))
-    )
-    (property "Footprint" "" (id 2) (at 89.8652 64.77 0)
+    (property "Value" "0.33uF" (id 1) (at 92.71 62.2299 0)
+      (effects (font (size 1.27 1.27)) (justify left))
+    )
+    (property "Footprint" "Resistor_THT:R_Axial_DIN0207_L6.3mm_D2.5mm_P2.54mm_Vertical" (id 2) (at 89.8652 64.77 0)
       (effects (font (size 1.27 1.27)) hide)
     )
@@
       (effects (font (size 1.27 1.27)) (justify left))
     )
-    (property "Footprint" "" (id 2) (at 147.0152 64.77 0)
+    (property "Footprint" "Capacitor_THT:C_Disc_D3.0mm_W2.0mm_P2.50mm" (id 2) (at 147.0152 64.77 0)
       (effects (font (size 1.27 1.27)) hide)
     )
@@
       (effects (font (size 1.27 1.27)) (justify left))
     )
-    (property "Value" "R" (id 1) (at 105.41 115.5699 0)
-      (effects (font (size 1.27 1.27)) (justify left))
-    )
-    (property "Footprint" "" (id 2) (at 101.092 114.3 90)
+    (property "Value" "1kohm" (id 1) (at 105.41 115.5699 0)
+      (effects (font (size 1.27 1.27)) (justify left))
+    )
+    (property "Footprint" "Resistor_THT:R_Axial_DIN0207_L6.3mm_D2.5mm_P7.62mm_Horizontal" (id 2) (at 101.092 114.3 90)
       (effects (font (size 1.27 1.27)) hide)
     )
@@
     (property "Reference" "D1" (id 0) (at 96.52 104.4575 0))
     (property "Value" "LED" (id 1) (at 99.06 104.4575 0))
-    (property "Footprint" "" (id 2) (at 102.87 102.87 0)
+    (property "Footprint" "LED_THT:LED_D4.0mm" (id 2) (at 102.87 102.87 0)
       (effects (font (size 1.27 1.27)) hide)
     )
@@
       (effects (font (size 1.27 1.27)) (justify left))
     )
-    (property "Footprint" "" (id 2) (at 246.38 100.33 0)
+    (property "Footprint" "TerminalBlock_Phoenix:TerminalBlock_Phoenix_MKDS-1,5-2-5.08_1x02_P5.08mm_Horizontal" (id 2) (at 246.38 100.33 0)
       (effects (font (size 1.27 1.27)) hide)
     )
@@
       (effects (font (size 1.27 1.27)) (justify left))
     )
-    (property "Footprint" "" (id 2) (at 110.1852 64.77 0)
+    (property "Footprint" "Capacitor_THT:C_Disc_D3.0mm_W2.0mm_P2.50mm" (id 2) (at 110.1852 64.77 0)
       (effects (font (size 1.27 1.27)) hide)
     )
@@
       (effects (font (size 1.27 1.27)) (justify left))
     )
-    (property "Footprint" "" (id 2) (at 172.72 100.33 0)
+    (property "Footprint" "TerminalBlock_Phoenix:TerminalBlock_Phoenix_MKDS-1,5-2-5.08_1x02_P5.08mm_Horizontal" (id 2) (at 172.72 100.33 0)
       (effects (font (size 1.27 1.27)) hide)
     )
@@
       (effects (font (size 1.27 1.27)) (justify left))
     )
-    (property "Value" "0.50uF" (id 1) (at 129.54 62.2299 0)
-      (effects (font (size 1.27 1.27)) (justify left))
-    )
-    (property "Footprint" "" (id 2) (at 126.6952 64.77 0)
+    (property "Value" "0.33uF" (id 1) (at 129.54 62.2299 0)
+      (effects (font (size 1.27 1.27)) (justify left))
+    )
+    (property "Footprint" "Capacitor_THT:C_Disc_D4.7mm_W2.5mm_P5.00mm" (id 2) (at 126.6952 64.77 0)
       (effects (font (size 1.27 1.27)) hide)
     )
@@
     )
     (path "/5129725e-4a4c-4676-b589-fa4f0f0e0f3e"
-      (reference "C1") (unit 1) (value "0.50uF") (footprint "")
+      (reference "C1") (unit 1) (value "0.33uF") (footprint "Resistor_THT:R_Axial_DIN0207_L6.3mm_D2.5mm_P2.54mm_Vertical")
     )
     (path "/c4e7cdf1-0468-447a-9fb2-cac1b5e5f41b"
-      (reference "C2") (unit 1) (value "0.50uF") (footprint "")
+      (reference "C2") (unit 1) (value "0.33uF") (footprint "Capacitor_THT:C_Disc_D4.7mm_W2.5mm_P5.00mm")
     )
     (path "/a2924c94-753f-47f3-af6a-4610f01a37b4"
-      (reference "C3") (unit 1) (value "0.1uF") (footprint "")
+      (reference "C3") (unit 1) (value "0.1uF") (footprint "Capacitor_THT:C_Disc_D3.0mm_W2.0mm_P2.50mm")
     )
     (path "/821f2bc8-6e7c-47e0-a40a-12b032c6db26"
-      (reference "C4") (unit 1) (value "0.1uF") (footprint "")
+      (reference "C4") (unit 1) (value "0.1uF") (footprint "Capacitor_THT:C_Disc_D3.0mm_W2.0mm_P2.50mm")
     )
     (path "/8d831f1d-717d-41b3-bb1b-c950ed23867e"
-      (reference "D1") (unit 1) (value "LED") (footprint "")
+      (reference "D1") (unit 1) (value "LED") (footprint "LED_THT:LED_D4.0mm")
     )
     (path "/0098889b-2a7f-4b25-8ecc-0c0f54924546"
-      (reference "D2") (unit 1) (value "LED") (footprint "")
+      (reference "D2") (unit 1) (value "LED") (footprint "LED_THT:LED_D4.0mm")
     )
     (path "/c2b901cd-ed8b-47be-8e02-5342a37f798a"
-      (reference "J1") (unit 1) (value "Screw_Terminal_01x02") (footprint "")
+      (reference "J1") (unit 1) (value "Screw_Terminal_01x02") (footprint "TerminalBlock_Phoenix:TerminalBlock_Phoenix_MKDS-1,5-2-5.08_1x02_P5.08mm_Horizontal")
     )
     (path "/39b14eb4-3585-44e1-abb0-33e10680d56a"
-      (reference "J2") (unit 1) (value "Screw_Terminal_01x02") (footprint "")
+      (reference "J2") (unit 1) (value "Screw_Terminal_01x02") (footprint "TerminalBlock_Phoenix:TerminalBlock_Phoenix_MKDS-1,5-2-5.08_1x02_P5.08mm_Horizontal")
     )
     (path "/91b87533-ea72-4aed-a93e-93176f2c27ad"
-      (reference "J3") (unit 1) (value "Screw_Terminal_01x02") (footprint "")
+      (reference "J3") (unit 1) (value "Screw_Terminal_01x02") (footprint "TerminalBlock_Phoenix:TerminalBlock_Phoenix_MKDS-1,5-2-5.08_1x02_P5.08mm_Horizontal")
     )
     (path "/3fecf9b7-f839-4eb7-b1a4-b4484ecd0148"
-      (reference "R1") (unit 1) (value "330ohm") (footprint "")
+      (reference "R1") (unit 1) (value "330ohm") (footprint "Resistor_THT:R_Axial_DIN0204_L3.6mm_D1.6mm_P5.08mm_Horizontal")
     )
     (path "/83102287-0dd5-4bec-875a-5836f4f05be9"
-      (reference "R2") (unit 1) (value "R") (footprint "")
+      (reference "R2") (unit 1) (value "1kohm") (footprint "Resistor_THT:R_Axial_DIN0207_L6.3mm_D2.5mm_P7.62mm_Horizontal")
     )
     (path "/1bfc539d-8a1c-423e-9ec9-1393433bbadd"
-      (reference "U1") (unit 1) (value "L7809") (footprint "")
+      (reference "U1") (unit 1) (value "L7809") (footprint "Package_TO_SOT_THT:TO-220-3_Vertical")
     )
     (path "/4573700a-5025-400f-bbfa-d09da177ed00"
-      (reference "U2") (unit 1) (value "L7805") (footprint "")
-    )
-  )
+      (reference "U2") (unit 1) (value "L7805") (footprint "Package_TO_SOT_THT:TO-220-3_Vertical")
+    )
+  )

Commit message: 08/01/23 sistemato i componenti nella pcb
Parts:
- C1: footprint Resistor_THT:R_Axial_DIN0207_L6.3mm_D2.5mm_P2.54mm_Vertical -> Capacitor_THT:C_Disc_D4.7mm_W2.5mm_P5.00mm
Changed lines of the file:
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@@
     (pin "1")
-  )
-  (symbol (lib_id "Device:C") (at 88.9 60.96 0) (unit 1)
-    (in_bom yes) (on_board yes) (fields_autoplaced)
-    (property "Reference" "C1" (id 0) (at 92.71 59.6899 0)
-      (effects (font (size 1.27 1.27)) (justify left))
-    )
-    (property "Value" "0.33uF" (id 1) (at 92.71 62.2299 0)
-      (effects (font (size 1.27 1.27)) (justify left))
-    )
-    (property "Footprint" "Resistor_THT:R_Axial_DIN0207_L6.3mm_D2.5mm_P2.54mm_Vertical" (id 2) (at 89.8652 64.77 0)
-      (effects (font (size 1.27 1.27)) hide)
-    )
-    (property "Datasheet" "~" (id 3) (at 88.9 60.96 0)
-      (effects (font (size 1.27 1.27)) hide)
-    )
-    (pin "1")
-    (pin "2")
   )
   (symbol (lib_id "power:PWR_FLAG") (at 104.14 72.39 180) (unit 1)
@@
     (pin "2")
   )
+  (symbol (lib_id "Device:C") (at 88.9 60.96 0) (unit 1)
+    (in_bom yes) (on_board yes)
+    (property "Reference" "C1" (id 0) (at 92.71 59.6899 0)
+      (effects (font (size 1.27 1.27)) (justify left))
+    )
+    (property "Value" "0.33uF" (id 1) (at 92.71 62.2299 0)
+      (effects (font (size 1.27 1.27)) (justify left))
+    )
+    (property "Footprint" "Capacitor_THT:C_Disc_D4.7mm_W2.5mm_P5.00mm" (id 2) (at 89.8652 64.77 0)
+      (effects (font (size 1.27 1.27)) hide)
+    )
+    (property "Datasheet" "~" (id 3) (at 88.9 60.96 0)
+      (effects (font (size 1.27 1.27)) hide)
+    )
+    (pin "1")
+    (pin "2")
+  )
   (symbol (lib_id "power:+12V") (at 165.1 100.33 0) (unit 1)
     (in_bom yes) (on_board yes) (fields_autoplaced)
@@
       (reference "#PWR0108") (unit 1) (value "GND") (footprint "")
     )
-    (path "/5129725e-4a4c-4676-b589-fa4f0f0e0f3e"
-      (reference "C1") (unit 1) (value "0.33uF") (footprint "Resistor_THT:R_Axial_DIN0207_L6.3mm_D2.5mm_P2.54mm_Vertical")
+    (path "/a42adc56-432c-4050-9686-ea4a9a7f3ca4"
+      (reference "C1") (unit 1) (value "0.33uF") (footprint "Capacitor_THT:C_Disc_D4.7mm_W2.5mm_P5.00mm")
     )
     (path "/c4e7cdf1-0468-447a-9fb2-cac1b5e5f41b"
