File: learn/Two_phese_bipolar_stepper_motor/Two_phese_bipolar_stepper_motor.kicad_pcb (KiCad board)
At the start: 2 copper layers, 21 parts, among them J1 Screw_Terminal_01x02, J2 Screw_Terminal_01x02, J3 Screw_Terminal_01x12, J4 Screw_Terminal_01x04, U1 L297, U2 L298N

Commit message: 12/06/2023 make a pcb
Parts:
- moved J1 107.2 mm to (143.2, 57.5)
- moved J2 107.1 mm to (126.0, 57.6)
- moved J4 96.7 mm to (136.5, 128.1)
- moved C4 91.2 mm to (136.7, 74.5)
- moved J3 90.1 mm to (181.4, 115.4)
- moved R1 85.9 mm to (152.9, 90.4)
- moved C2 84.6 mm to (150.4, 74.2)
- moved Rs2 84.3 mm to (138.9, 103.4)
- moved Rs1 84.3 mm to (149.1, 103.4)
- moved U1 82.8 mm to (168.9, 93.5)
- moved D1 82.8 mm to (157.7, 101.3)
- moved D2 82.8 mm to (157.7, 108.2)
- moved D3 82.8 mm to (157.7, 115.1)
- moved D4 82.8 mm to (157.7, 122.0)
- moved D5 81.9 mm to (115.5, 101.2)
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Other:
- board outline added: 73.7 x 81 mm

Commit message: two_phese: made PCB
Parts:
- added REF**: MountingHole_2.5mm, MountingHole:MountingHole_2.5mm, F.Cu at (181.7, 129.0)
- added REF**: MountingHole_2.5mm, MountingHole:MountingHole_2.5mm, F.Cu at (117.2, 56.8)
- added REF**: MountingHole_2.5mm, MountingHole:MountingHole_2.5mm, F.Cu at (180.9, 56.8)
- added REF**: MountingHole_2.5mm, MountingHole:MountingHole_2.5mm, F.Cu at (117.5, 129.0)
- moved J3 5.28 mm to (181.4, 120.7)
- moved J2 3.91 mm to (129.9, 57.5)
Changed lines of the file:
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@@
   )
   (setup
+    (stackup
+      (layer "F.SilkS" (type "Top Silk Screen"))
+      (layer "F.Paste" (type "Top Solder Paste"))
+      (layer "F.Mask" (type "Top Solder Mask") (thickness 0.01))
+      (layer "F.Cu" (type "copper") (thickness 0.035))
+      (layer "dielectric 1" (type "core") (thickness 1.51) (material "FR4") (epsilon_r 4.5) (loss_tangent 0.02))
+      (layer "B.Cu" (type "copper") (thickness 0.035))
+      (layer "B.Mask" (type "Bottom Solder Mask") (thickness 0.01))
+      (layer "B.Paste" (type "Bottom Solder Paste"))
+      (layer "B.SilkS" (type "Bottom Silk Screen"))
+      (copper_finish "None")
+      (dielectric_constraints no)
+    )
     (pad_to_mask_clearance 0)
     (pcbplotparams
@@
     )
   )
+  (footprint "MountingHole:MountingHole_2.5mm" (layer "F.Cu")
+    (at 181.7 129.025)
+    (descr "Mounting Hole 2.5mm, no annular")
+    (tags "mounting hole 2.5mm no annular")
+    (attr exclude_from_pos_files exclude_from_bom)
+    (fp_text reference "REF**" (at 0 -3.5) (layer "F.SilkS") hide
+        (effects (font (size 1 1) (thickness 0.15)))
+    )
+    (fp_text value "MountingHole_2.5mm" (at 0 3.5) (layer "F.Fab") hide
+        (effects (font (size 1 1) (thickness 0.15)))
+    )
+    (fp_text user "${REFERENCE}" (at 0 0) (layer "F.Fab")
+        (effects (font (size 1 1) (thickness 0.15)))
+    )
+    (fp_circle (center 0 0) (end 2.5 0)
+      (stroke (width 0.15) (type solid)) (fill none) (layer "Cmts.User"))
+    (fp_circle (center 0 0) (end 2.75 0)
+      (stroke (width 0.05) (type solid)) (fill none) (layer "F.CrtYd"))
+    (pad "" np_thru_hole circle (at 0 0) (size 2.5 2.5) (drill 2.5) (layers "F&B.Cu" "*.Mask"))
+  )
   (footprint "Diode_THT:D_DO-27_P15.24mm_Horizontal" (layer "F.Cu")
     (at 157.734 121.99)
@@
     (property "ki_keywords" "screw terminal")
     (attr through_hole)
-    (fp_text reference "J1" (at 2.54 -6.26) (layer "F.SilkS")
-        (effects (font (size 1 1) (thickness 0.15)))
-    )
-    (fp_text value "Screw_Terminal_01x02" (at 2.54 5.66) (layer "F.Fab")
+    (fp_text reference "J1" (at 2.54 -6.26) (layer "F.SilkS") hide
+        (effects (font (size 1 1) (thickness 0.15)))
+    )
+    (fp_text value "Screw_Terminal_01x02" (at 2.54 5.66) (layer "F.Fab") hide
         (effects (font (size 1 1) (thickness 0.15)))
     )
@@
     )
   )
+  (footprint "MountingHole:MountingHole_2.5mm" (layer "F.Cu")
+    (at 117.175 56.75)
+    (descr "Mounting Hole 2.5mm, no annular")
+    (tags "mounting hole 2.5mm no annular")
+    (attr exclude_from_pos_files exclude_from_bom)
+    (fp_text reference "REF**" (at 0 -3.5) (layer "F.SilkS") hide
+        (effects (font (size 1 1) (thickness 0.15)))
+    )
+    (fp_text value "MountingHole_2.5mm" (at 0 3.5) (layer "F.Fab") hide
+        (effects (font (size 1 1) (thickness 0.15)))
+    )
+    (fp_text user "${REFERENCE}" (at 0 0) (layer "F.Fab")
+        (effects (font (size 1 1) (thickness 0.15)))
+    )
+    (fp_circle (center 0 0) (end 2.5 0)
+      (stroke (width 0.15) (type solid)) (fill none) (layer "Cmts.User"))
+    (fp_circle (center 0 0) (end 2.75 0)
+      (stroke (width 0.05) (type solid)) (fill none) (layer "F.CrtYd"))
+    (pad "" np_thru_hole circle (at 0 0) (size 2.5 2.5) (drill 2.5) (layers "F&B.Cu" "*.Mask"))
+  )
   (footprint "Diode_THT:D_DO-27_P15.24mm_Horizontal" (layer "F.Cu")
     (at 115.51 121.92)
@@
       (rotate (xyz 0 0 0))
     )
+  )
+  (footprint "MountingHole:MountingHole_2.5mm" (layer "F.Cu")
+    (at 180.95 56.75)
+    (descr "Mounting Hole 2.5mm, no annular")
+    (tags "mounting hole 2.5mm no annular")
+    (attr exclude_from_pos_files exclude_from_bom)
+    (fp_text reference "REF**" (at 0 -3.5) (layer "F.SilkS") hide
+        (effects (font (size 1 1) (thickness 0.15)))
+    )
+    (fp_text value "MountingHole_2.5mm" (at 0 3.5) (layer "F.Fab") hide
+        (effects (font (size 1 1) (thickness 0.15)))
+    )
+    (fp_text user "${REFERENCE}" (at 0 0) (layer "F.Fab")
+        (effects (font (size 1 1) (thickness 0.15)))
+    )
+    (fp_circle (center 0 0) (end 2.5 0)
+      (stroke (width 0.15) (type solid)) (fill none) (layer "Cmts.User"))
+    (fp_circle (center 0 0) (end 2.75 0)
+      (stroke (width 0.05) (type solid)) (fill none) (layer "F.CrtYd"))
+    (pad "" np_thru_hole circle (at 0 0) (size 2.5 2.5) (drill 2.5) (layers "*.Cu" "*.Mask"))
   )
   (footprint "Package_DIP:DIP-20_W7.62mm_LongPads" (layer "F.Cu")
@@
     )
   )
+  (footprint "MountingHole:MountingHole_2.5mm" (layer "F.Cu")
+    (at 117.5 129.025)
+    (descr "Mounting Hole 2.5mm, no annular")
+    (tags "mounting hole 2.5mm no annular")
+    (attr exclude_from_pos_files exclude_from_bom)
+    (fp_text reference "REF**" (at 0 -3.5) (layer "F.SilkS") hide
+        (effects (font (size 1 1) (thickness 0.15)))
+    )
+    (fp_text value "MountingHole_2.5mm" (at 0 3.5) (layer "F.Fab") hide
+        (effects (font (size 1 1) (thickness 0.15)))
+    )
+    (fp_text user "${REFERENCE}" (at 0 0) (layer "F.Fab")
+        (effects (font (size 1 1) (thickness 0.15)))
+    )
+    (fp_circle (center 0 0) (end 2.5 0)
+      (stroke (width 0.15) (type solid)) (fill none) (layer "Cmts.User"))
+    (fp_circle (center 0 0) (end 2.75 0)
+      (stroke (width 0.05) (type solid)) (fill none) (layer "F.CrtYd"))
+    (pad "" np_thru_hole circle (at 0 0) (size 2.5 2.5) (drill 2.5) (layers "F&B.Cu" "*.Mask"))
+  )
   (footprint "TerminalBlock_Phoenix:TerminalBlock_Phoenix_MKDS-1,5-2-5.08_1x02_P5.08mm_Horizontal" (layer "F.Cu")
-    (at 126.035 57.585 180)
+    (at 129.945 57.545 180)
     (descr "Terminal Block Phoenix MKDS-1,5-2-5.08, 2 pins, pitch 5.08mm, size 10.2x9.8mm^2, drill diamater 1.3mm, pad diameter 2.6mm, see http://www.farnell.com/datasheets/100425.pdf, script-generated using https://github.com/pointhi/kicad-footprint-generator/scripts/TerminalBlock_Phoenix")
     (tags "THT Terminal Block Phoenix MKDS-1,5-2-5.08 pitch 5.08mm size 10.2x9.8mm^2 drill 1.3mm pad 2.6mm")
@@
     (property "ki_keywords" "screw terminal")
     (attr through_hole)
-    (fp_text reference "J2" (at 2.54 -6.26) (layer "F.SilkS")
-        (effects (font (size 1 1) (thickness 0.15)))
-    )
-    (fp_text value "Screw_Terminal_01x02" (at 2.54 5.66) (layer "F.Fab")
+    (fp_text reference "J2" (at 2.54 -6.26) (layer "F.SilkS") hide
+        (effects (font (size 1 1) (thickness 0.15)))
+    )
+    (fp_text value "Screw_Terminal_01x02" (at 2.54 5.66) (layer "F.Fab") hide
         (effects (font (size 1 1) (thickness 0.15)))
     )
@@
   )
   (footprint "TerminalBlock_Phoenix:TerminalBlock_Phoenix_MKDS-1,5-12_1x12_P5.00mm_Horizontal" (layer "F.Cu")
-    (at 181.44 115.42 90)
+    (at 181.45 120.7 90)
     (descr "Terminal Block Phoenix MKDS-1,5-12, 12 pins, pitch 5mm, size 60x9.8mm^2, drill diamater 1.3mm, pad diameter 2.6mm, see http://www.farnell.com/datasheets/100425.pdf, script-generated using https://github.com/pointhi/kicad-footprint-generator/scripts/TerminalBlock_Phoenix")
     (tags "THT Terminal Block Phoenix MKDS-1,5-12 pitch 5mm size 60x9.8mm^2 drill 1.3mm pad 2.6mm")
@@
     (property "ki_keywords" "screw terminal")
     (attr through_hole)
-    (fp_text reference "J3" (at 27.5 -6.26 90) (layer "F.SilkS")
-        (effects (font (size 1 1) (thickness 0.15)))
-    )
-    (fp_text value "Screw_Terminal_01x12" (at 27.5 5.66 90) (layer "F.Fab")
-        (effects (font (size 1 1) (thickness 0.15)))
-    )
+    (fp_text reference "J3" (at 27.5 -6.26 90) (layer "F.SilkS") hide
+        (effects (font (size 1 1) (thickness 0.15)))
+    )
+    (fp_text value "Screw_Terminal_01x12" (at 27.5 5.66 90) (layer "F.Fab") hide
+        (effects (font (size 1 1) (thickness 0.15)))
+    )
