File: learn/Two_phese_bipolar_stepper_motor/Two_phese_bipolar_stepper_motor.kicad_sch (KiCad schematic)
At the start: 21 parts, among them J1 Screw_Terminal_01x02, J2 Screw_Terminal_01x02, J3 Screw_Terminal_01x12, J4 Screw_Terminal_01x04, U1 L297, U2 L298N

Commit message: 04/06/2023 etichettature
Other:
- note added: "Control signal connector"
- note added: "Logic power supply"
- note added: "Logic power supply connector"
- note added: "Main control unit"
- note added: "Motor power supply"
- note added: "Motor power supply connector"
- note added: "Motor windings connector"
- moved on the sheet: J2, Rs1, Rs2

Commit message: 04/06/2023 inizio assegnazione impronte
Parts:
- C1: footprint (none) -> Capacitor_THT:C_Rect_L10.0mm_W3.0mm_P7.50mm_FKS3_FKP3
- C2, C3: footprint (none) -> Capacitor_THT:C_Rect_L7.5mm_W6.5mm_P5.00mm
- C4: footprint (none) -> Capacitor_THT:CP_Radial_D13.0mm_P5.00mm
- D1, D2, D3, D4, D5, D6, D7, D8: footprint (none) -> Diode_THT:D_DO-27_P15.24mm_Horizontal
Changed lines of the file:
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@@
       (effects (font (size 1.27 1.27)) (justify left))
     )
-    (property "Footprint" "" (at 207.01 104.14 0)
+    (property "Footprint" "Diode_THT:D_DO-27_P15.24mm_Horizontal" (at 207.01 104.14 0)
       (effects (font (size 1.27 1.27)) hide)
     )
@@
       (effects (font (size 1.27 1.27)) (justify left))
     )
-    (property "Footprint" "" (at 191.77 129.54 0)
+    (property "Footprint" "Diode_THT:D_DO-27_P15.24mm_Horizontal" (at 191.77 129.54 0)
       (effects (font (size 1.27 1.27)) hide)
     )
@@
       (effects (font (size 1.27 1.27)) (justify left))
     )
-    (property "Footprint" "" (at 191.77 104.14 0)
+    (property "Footprint" "Diode_THT:D_DO-27_P15.24mm_Horizontal" (at 191.77 104.14 0)
       (effects (font (size 1.27 1.27)) hide)
     )
@@
       (effects (font (size 1.27 1.27)) (justify left))
     )
-    (property "Footprint" "" (at 131.7752 46.99 0)
+    (property "Footprint" "Capacitor_THT:CP_Radial_D13.0mm_P5.00mm" (at 131.7752 46.99 0)
       (effects (font (size 1.27 1.27)) hide)
     )
@@
       (effects (font (size 1.27 1.27)) (justify left))
     )
-    (property "Footprint" "" (at 184.15 129.54 0)
+    (property "Footprint" "Diode_THT:D_DO-27_P15.24mm_Horizontal" (at 184.15 129.54 0)
       (effects (font (size 1.27 1.27)) hide)
     )
@@
       (effects (font (size 1.27 1.27)) (justify left))
     )
-    (property "Footprint" "" (at 207.01 129.54 0)
+    (property "Footprint" "Diode_THT:D_DO-27_P15.24mm_Horizontal" (at 207.01 129.54 0)
       (effects (font (size 1.27 1.27)) hide)
     )
@@
       (effects (font (size 1.27 1.27)) (justify left))
     )
-    (property "Footprint" "" (at 184.15 104.14 0)
+    (property "Footprint" "Diode_THT:D_DO-27_P15.24mm_Horizontal" (at 184.15 104.14 0)
       (effects (font (size 1.27 1.27)) hide)
     )
@@
       (effects (font (size 1.27 1.27)) (justify left))
     )
-    (property "Footprint" "" (at 199.39 129.54 0)
+    (property "Footprint" "Diode_THT:D_DO-27_P15.24mm_Horizontal" (at 199.39 129.54 0)
       (effects (font (size 1.27 1.27)) hide)
     )
@@
       (effects (font (size 1.27 1.27)) (justify left))
     )
-    (property "Footprint" "" (at 199.39 104.14 0)
+    (property "Footprint" "Diode_THT:D_DO-27_P15.24mm_Horizontal" (at 199.39 104.14 0)
       (effects (font (size 1.27 1.27)) hide)
     )
@@
       (effects (font (size 1.27 1.27)) (justify left))
     )
-    (property "Footprint" "" (at 84.7852 48.26 0)
+    (property "Footprint" "Capacitor_THT:C_Rect_L10.0mm_W3.0mm_P7.50mm_FKS3_FKP3" (at 84.7852 48.26 0)
       (effects (font (size 1.27 1.27)) hide)
     )
@@
       (effects (font (size 1.27 1.27)) (justify left))
     )
-    (property "Footprint" "" (at 149.5552 46.99 0)
+    (property "Footprint" "Capacitor_THT:C_Rect_L7.5mm_W6.5mm_P5.00mm" (at 149.5552 46.99 0)
       (effects (font (size 1.27 1.27)) hide)
     )
@@
       (effects (font (size 1.27 1.27)) (justify left))
     )
-    (property "Footprint" "" (at 107.6452 48.26 0)
-      (effects (font (size 1.27 1.27)) hide)
-    )
+    (property "Footprint" "Capacitor_THT:C_Rect_L7.5mm_W6.5mm_P5.00mm" (at 107.6452 48.26 0)
+      (effects (font (size 1.27 1.27)) hide)
+    )

Commit message: 10/06/2023 write the footprint
Parts:
- J1, J2: footprint (none) -> TerminalBlock_Phoenix:TerminalBlock_Phoenix_MKDS-1,5-2-5.08_1x02_P5.08mm_Horizontal
- J3: footprint (none) -> TerminalBlock_Phoenix:TerminalBlock_Phoenix_MKDS-1,5-12_1x12_P5.00mm_Horizontal
- J4: footprint (none) -> TerminalBlock_Phoenix:TerminalBlock_Phoenix_MKDS-1,5-4_1x04_P5.00mm_Horizontal
- R1: footprint (none) -> Resistor_THT:R_Axial_DIN0922_L20.0mm_D9.0mm_P25.40mm_Horizontal
- Rs1, Rs2: footprint (none) -> Resistor_THT:R_Axial_DIN0414_L11.9mm_D4.5mm_P15.24mm_Horizontal
- U1: footprint (none) -> Package_DIP:DIP-20_W7.62mm_LongPads
Changed lines of the file:
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@@
       (effects (font (size 1.27 1.27)) (justify left))
     )
-    (property "Footprint" "" (at 177.8 53.34 0)
+    (property "Footprint" "TerminalBlock_Phoenix:TerminalBlock_Phoenix_MKDS-1,5-2-5.08_1x02_P5.08mm_Horizontal" (at 177.8 53.34 0)
       (effects (font (size 1.27 1.27)) hide)
     )
@@
       (effects (font (size 1.27 1.27)))
     )
-    (property "Footprint" "" (at 72.39 118.11 0)
+    (property "Footprint" "TerminalBlock_Phoenix:TerminalBlock_Phoenix_MKDS-1,5-12_1x12_P5.00mm_Horizontal" (at 72.39 118.11 0)
       (effects (font (size 1.27 1.27)) hide)
     )
@@
       (effects (font (size 1 1)) (justify left))
     )
-    (property "Footprint" "" (at 66.802 161.29 90)
+    (property "Footprint" "Resistor_THT:R_Axial_DIN0414_L11.9mm_D4.5mm_P15.24mm_Horizontal" (at 66.802 161.29 90)
       (effects (font (size 1.27 1.27)) hide)
     )
@@
       (effects (font (size 1.27 1.27)) (justify left))
     )
-    (property "Footprint" "" (at 177.8 30.48 0)
+    (property "Footprint" "TerminalBlock_Phoenix:TerminalBlock_Phoenix_MKDS-1,5-2-5.08_1x02_P5.08mm_Horizontal" (at 177.8 30.48 0)
       (effects (font (size 1.27 1.27)) hide)
     )
@@
       (effects (font (size 1.27 1.27)))
     )
-    (property "Footprint" "" (at 90.17 39.878 90)
+    (property "Footprint" "Resistor_THT:R_Axial_DIN0922_L20.0mm_D9.0mm_P25.40mm_Horizontal" (at 90.17 39.878 90)
       (effects (font (size 1.27 1.27)) hide)
     )
@@
       (effects (font (size 1.27 1.27)) (justify left))
     )
-    (property "Footprint" "" (at 223.52 115.57 0)
+    (property "Footprint" "TerminalBlock_Phoenix:TerminalBlock_Phoenix_MKDS-1,5-4_1x04_P5.00mm_Horizontal" (at 223.52 115.57 0)
       (effects (font (size 1.27 1.27)) hide)
     )
@@
       (effects (font (size 1 1)) (justify left))
     )
-    (property "Footprint" "" (at 76.962 161.29 90)
+    (property "Footprint" "Resistor_THT:R_Axial_DIN0414_L11.9mm_D4.5mm_P15.24mm_Horizontal" (at 76.962 161.29 90)
       (effects (font (size 1.27 1.27)) hide)
     )
@@
       (effects (font (size 1.27 1.27)) (justify left))
     )
-    (property "Footprint" "" (at 111.76 101.6 0)
-      (effects (font (size 1.27 1.27)) hide)
-    )
+    (property "Footprint" "Package_DIP:DIP-20_W7.62mm_LongPads" (at 111.76 101.6 0)
+      (effects (font (size 1.27 1.27)) hide)
+    )

Commit message: Two_phase: print the wire
Connections:
- net VSS is gone; now on net VS: C2.1, J2.1 (Pin_1), R1.2, U1.12 (Vs), U2.9 (Vss)
Changed lines of the file:
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@@
   (junction (at 199.39 99.06) (diameter 0) (color 0 0 0 0)
   )
+  (junction (at 99.06 36.83) (diameter 0) (color 0 0 0 0)
+  )
   (junction (at 199.39 134.62) (diameter 0) (color 0 0 0 0)
   )
@@
   )
   (junction (at 139.7 36.83) (diameter 0) (color 0 0 0 0)
-  )
-  (junction (at 99.06 36.83) (diameter 0) (color 0 0 0 0)
   )
   (junction (at 95.25 48.26) (diameter 0) (color 0 0 0 0)
@@
     )
   )
-  (symbol (lib_id "power:VSS") (at 161.29 99.06 0) (unit 1)
-    (in_bom yes) (on_board yes) (dnp no)
-    (property "Reference" "#PWR0111" (at 161.29 102.87 0)
-      (effects (font (size 1.27 1.27)) hide)
-    )
-    (property "Value" "VSS" (at 160.02 95.25 0)
-      (effects (font (size 0.9 0.9)) (justify left))
-    )
-    (property "Footprint" "" (at 161.29 99.06 0)
-      (effects (font (size 1.27 1.27)) hide)
-    )
-    (property "Datasheet" "" (at 161.29 99.06 0)
-      (effects (font (size 1.27 1.27)) hide)
-    )
-    (pin "1")
-    (instances
-      (project "Two_phese_bipolar_stepper_motor"
-        (path "/0fc27e7e-5941-43c9-87ba-c9c5a2c90ad0"
-          (reference "#PWR0111") (unit 1)
-        )
-      )
-    )
-  )
   (symbol (lib_id "power:GND") (at 95.25 50.8 0) (unit 1)
     (in_bom yes) (on_board yes) (dnp no) (fields_autoplaced)
@@
     )
   )
+  (symbol (lib_id "power:VS") (at 99.06 36.83 0) (unit 1)
+    (in_bom yes) (on_board yes) (dnp no) (fields_autoplaced)
+    (property "Reference" "#PWR02" (at 93.98 40.64 0)
+      (effects (font (size 1.27 1.27)) hide)
+    )
+    (property "Value" "VS" (at 99.06 31.75 0)
+      (effects (font (size 1.27 1.27)))
+    )
+    (property "Footprint" "" (at 99.06 36.83 0)
+      (effects (font (size 1.27 1.27)) hide)
+    )
+    (property "Datasheet" "" (at 99.06 36.83 0)
+      (effects (font (size 1.27 1.27)) hide)
+    )
+    (pin "1")
+    (instances
+      (project "Two_phese_bipolar_stepper_motor"
+        (path "/0fc27e7e-5941-43c9-87ba-c9c5a2c90ad0"
+          (reference "#PWR02") (unit 1)
+        )
+      )
+    )
+  )
+  (symbol (lib_id "power:VS") (at 161.29 99.06 0) (unit 1)
+    (in_bom yes) (on_board yes) (dnp no) (fields_autoplaced)
+    (property "Reference" "#PWR04" (at 156.21 102.87 0)
+      (effects (font (size 1.27 1.27)) hide)
+    )
+    (property "Value" "VS" (at 161.29 93.98 0)
+      (effects (font (size 1.27 1.27)))
+    )
+    (property "Footprint" "" (at 161.29 99.06 0)
+      (effects (font (size 1.27 1.27)) hide)
+    )
+    (property "Datasheet" "" (at 161.29 99.06 0)
+      (effects (font (size 1.27 1.27)) hide)
+    )
+    (pin "1")
+    (instances
+      (project "Two_phese_bipolar_stepper_motor"
+        (path "/0fc27e7e-5941-43c9-87ba-c9c5a2c90ad0"
+          (reference "#PWR04") (unit 1)
+        )
+      )
+    )
+  )
   (symbol (lib_id "power:PWR_FLAG") (at 105.41 36.83 0) (unit 1)
     (in_bom yes) (on_board yes) (dnp no)
@@
     )
   )
-  (symbol (lib_id "power:VSS") (at 99.06 36.83 0) (unit 1)
-    (in_bom yes) (on_board yes) (dnp no) (fields_autoplaced)
-    (property "Reference" "#PWR0109" (at 99.06 40.64 0)
-      (effects (font (size 1.27 1.27)) hide)
-    )
-    (property "Value" "VSS" (at 99.06 31.75 0)
-      (effects (font (size 1.27 1.27)))
-    )
-    (property "Footprint" "" (at 99.06 36.83 0)
-      (effects (font (size 1.27 1.27)) hide)
-    )
-    (property "Datasheet" "" (at 99.06 36.83 0)
-      (effects (font (size 1.27 1.27)) hide)
-    )
-    (pin "1")
-    (instances
-      (project "Two_phese_bipolar_stepper_motor"
-        (path "/0fc27e7e-5941-43c9-87ba-c9c5a2c90ad0"
-          (reference "#PWR0109") (unit 1)
-        )
-      )
-    )
-  )
   (symbol (lib_id "power:GND") (at 86.36 105.41 0) (unit 1)
     (in_bom yes) (on_board yes) (dnp no) (fields_autoplaced)
@@
     )
   )
+  (symbol (lib_id "power:VS") (at 172.72 53.34 0) (unit 1)
+    (in_bom yes) (on_board yes) (dnp no) (fields_autoplaced)
+    (property "Reference" "#PWR01" (at 167.64 57.15 0)
+      (effects (font (size 1.27 1.27)) hide)
+    )
+    (property "Value" "VS" (at 172.72 48.26 0)
+      (effects (font (size 1.27 1.27)))
+    )
+    (property "Footprint" "" (at 172.72 53.34 0)
+      (effects (font (size 1.27 1.27)) hide)
+    )
+    (property "Datasheet" "" (at 172.72 53.34 0)
+      (effects (font (size 1.27 1.27)) hide)
+    )
+    (pin "1")
+    (instances
+      (project "Two_phese_bipolar_stepper_motor"
+        (path "/0fc27e7e-5941-43c9-87ba-c9c5a2c90ad0"
+          (reference "#PWR01") (unit 1)
+        )
+      )
+    )
+  )
   (symbol (lib_id "power:VS") (at 139.7 36.83 0) (unit 1)
     (in_bom yes) (on_board yes) (dnp no) (fields_autoplaced)
@@
         (path "/0fc27e7e-5941-43c9-87ba-c9c5a2c90ad0"
           (reference "D8") (unit 1)
-        )
-      )
-    )
-  )
-  (symbol (lib_id "power:VSS") (at 172.72 53.34 0) (unit 1)
-    (in_bom yes) (on_board yes) (dnp no) (fields_autoplaced)
-    (property "Reference" "#PWR0105" (at 172.72 57.15 0)
-      (effects (font (size 1.27 1.27)) hide)
-    )
-    (property "Value" "VSS" (at 172.72 48.26 0)
-      (effects (font (size 1.27 1.27)))
-    )
-    (property "Footprint" "" (at 172.72 53.34 0)
-      (effects (font (size 1.27 1.27)) hide)
-    )
-    (property "Datasheet" "" (at 172.72 53.34 0)
-      (effects (font (size 1.27 1.27)) hide)
-    )
-    (pin "1")
-    (instances
-      (project "Two_phese_bipolar_stepper_motor"
-        (path "/0fc27e7e-5941-43c9-87ba-c9c5a2c90ad0"
-          (reference "#PWR0105") (unit 1)
-        )
-      )
-    )
-  )
-  (symbol (lib_id "power:VSS") (at 123.19 97.79 0) (unit 1)
-    (in_bom yes) (on_board yes) (dnp no)
-    (property "Reference" "#PWR0115" (at 123.19 101.6 0)
-      (effects (font (size 1.27 1.27)) hide)
-    )
-    (property "Value" "VSS" (at 121.92 93.98 0)
-      (effects (font (size 0.9 0.9)) (justify left))
-    )
-    (property "Footprint" "" (at 123.19 97.79 0)
-      (effects (font (size 1.27 1.27)) hide)
-    )
-    (property "Datasheet" "" (at 123.19 97.79 0)
-      (effects (font (size 1.27 1.27)) hide)
-    )
-    (pin "1")
-    (instances
-      (project "Two_phese_bipolar_stepper_motor"
-        (path "/0fc27e7e-5941-43c9-87ba-c9c5a2c90ad0"
-          (reference "#PWR0115") (unit 1)
         )
       )
@@
         )
       )
+    )
+  )
+  (symbol (lib_id "power:VS") (at 123.19 97.79 0) (unit 1)
+    (in_bom yes) (on_board yes) (dnp no) (fields_autoplaced)
+    (property "Reference" "#PWR03" (at 118.11 101.6 0)
+      (effects (font (size 1.27 1.27)) hide)
+    )
+    (property "Value" "VS" (at 123.19 92.71 0)
+      (effects (font (size 1.27 1.27)))
+    )
+    (property "Footprint" "" (at 123.19 97.79 0)
+      (effects (font (size 1.27 1.27)) hide)
+    )
+    (property "Datasheet" "" (at 123.19 97.79 0)
+      (effects (font (size 1.27 1.27)) hide)
+    )
+    (pin "1")
+    (instances
+      (project "Two_phese_bipolar_stepper_motor"
+        (path "/0fc27e7e-5941-43c9-87ba-c9c5a2c90ad0"
+          (reference "#PWR03") (unit 1)
+        )
+      )
